Commit message: delete joint_2 for robot_control_setup

File: canopen_tests/urdf/robot_controller/robot_controller.macro.xacro (robot description, xacro)
@@ -51,5 +51,5 @@
         <limit lower="${-2*pi}" upper="${2*pi}" effort="10.0" velocity="0.5"/>
     </joint>
-    <joint name="${prefix}joint2" type="revolute">
+    <joint name="${prefix}joint2" type="fixed">
         <parent link="${prefix}link2"/>
         <child link="${prefix}link3"/>
